Commit message: controller works

File: rca_description/urdf/material.xacro (robot description, xacro)
@@ -1,5 +1,5 @@
 <?xml version="1.0"?>
 <robot xmlns:xacro="http://www.ros.org/wiki/xacro" >
-    <xacro:property name="PI" value="3.14159" />
+    <xacro:property name="PI" value="3.14159265359" />
     <xacro:property name="effort" value="30.0" />
     <xacro:property name="velocity" value="10.0" />

File: rca_description/urdf/rca_core.xacro (robot description, xacro)
@@ -6,5 +6,5 @@
         <xacro:default_inertial mass="3" />
         <visual>
-            <origin xyz="0.0 0.0 -0.065" rpy="0.0 0.0 ${pi}" />
+            <origin xyz="0.0 0.0 -0.065" rpy="0.0 0.0 ${PI}" />
             <geometry>
                 <mesh filename="package://rca_description/meshes/RCA_BASE_TOWER4URDF.stl"
@@ -14,5 +14,5 @@
         </visual>
         <collision>
-            <origin xyz="0.0 0.0 -0.065" rpy="0.0 0.0 ${pi}" />
+            <origin xyz="0.0 0.0 -0.065" rpy="0.0 0.0 ${PI}" />
             <geometry>
                 <mesh filename="package://rca_description/meshes/RCA_BASE_TOWER4URDF.stl"
@@ -24,5 +24,5 @@
         <xacro:default_inertial mass="0.5" />
         <visual>
-            <origin xyz="0.0 0.0 0" rpy="${pi/2} 0.0 ${-pi/2}" />
+            <origin xyz="0.0 0.0 0" rpy="${PI/2} 0.0 ${-PI/2}" />
             <geometry>
                 <mesh filename="package://rca_description/meshes/Waist.stl"
@@ -32,5 +32,5 @@
         </visual>
         <collision>
-            <origin xyz="0.0 0.0 0" rpy="${pi/2} 0.0 ${-pi/2}" />
+            <origin xyz="0.0 0.0 0" rpy="${PI/2} 0.0 ${-PI/2}" />
             <geometry>
                 <mesh filename="package://rca_description/meshes/Waist.stl"
@@ -42,5 +42,5 @@
         <xacro:default_inertial mass="0.3" />
         <visual>
-            <origin xyz="0.0 -0.001 0" rpy="${pi/2} 0 0" />
+            <origin xyz="0.0 -0.001 0" rpy="${PI/2} 0 0" />
             <geometry>
                 <mesh filename="package://rca_description/meshes/Arm_01.stl"
@@ -50,5 +50,5 @@
         </visual>
         <collision>
-            <origin xyz="0.0 -0.001 0" rpy="${pi/2} 0 0" />
+            <origin xyz="0.0 -0.001 0" rpy="${PI/2} 0 0" />
             <geometry>
                 <mesh filename="package://rca_description/meshes/Arm_01.stl"
@@ -60,5 +60,5 @@
         <xacro:default_inertial mass="0.3" />
         <visual>
-            <origin xyz="0 0.0018 0.035" rpy="${pi/2} 0 ${pi}" />
+            <origin xyz="0 0.0018 0.035" rpy="${PI/2} 0 ${PI}" />
             <geometry>
                 <mesh filename="package://rca_description/meshes/Arm_02.stl"
@@ -68,5 +68,5 @@
         </visual>
         <collision>
-            <origin xyz="0 0.0018 0.035" rpy="${pi/2} 0 ${pi}" />
+            <origin xyz="0 0.0018 0.035" rpy="${PI/2} 0 ${PI}" />
             <geometry>
                 <mesh filename="package://rca_description/meshes/Arm_02.stl"
@@ -78,5 +78,5 @@
         <xacro:default_inertial mass="0.2" />
         <visual>
-            <origin xyz="-0.0035 0 0.0015" rpy="${pi/2} 0 ${pi}" />
+            <origin xyz="-0.0035 0 0.0015" rpy="${PI/2} 0 ${PI}" />
             <geometry>
                 <mesh filename="package://rca_description/meshes/Arm_03.stl"
@@ -86,5 +86,5 @@
         </visual>
         <collision>
-            <origin xyz="-0.0035 0 0.0015" rpy="${pi/2} 0 ${pi}" />
+            <origin xyz="-0.0035 0 0.0015" rpy="${PI/2} 0 ${PI}" />
             <geometry>
                 <mesh filename="package://rca_description/meshes/Arm_03.stl"
@@ -96,5 +96,5 @@
         <xacro:default_inertial mass="0.2" />
         <visual>
-            <origin xyz="0.0095 0.005 0.063" rpy="0 0 ${-pi/2}" />
+            <origin xyz="0.0095 0.005 0.063" rpy="0 0 ${-PI/2}" />
             <geometry>
                 <mesh filename="package://rca_description/meshes/Gripper_base.stl"
@@ -104,5 +104,5 @@
         </visual>
         <collision>
-            <origin xyz="0.0095 0.005 0.063" rpy="0 0 ${-pi/2}" />
+            <origin xyz="0.0095 0.005 0.063" rpy="0 0 ${-PI/2}" />
             <geometry>
                 <mesh filename="package://rca_description/meshes/Gripper_base.stl"
@@ -114,5 +114,5 @@
         <xacro:default_inertial mass="0.1" />
         <visual>
-            <origin xyz="0 -0.003 -0.0065" rpy="${-pi/8} ${pi} 0" />
+            <origin xyz="0 -0.003 -0.0065" rpy="${-PI/8} ${PI} 0" />
             <geometry>
                 <mesh filename="package://rca_description/meshes/Gripper_1.stl"
@@ -122,5 +122,5 @@
         </visual>
         <collision>
-            <origin xyz="0 -0.003 -0.0065" rpy="${-pi/8} ${pi} 0" />
+            <origin xyz="0 -0.003 -0.0065" rpy="${-PI/8} ${PI} 0" />
             <geometry>
                 <mesh filename="package://rca_description/meshes/Gripper_1.stl"
@@ -132,5 +132,5 @@
         <xacro:default_inertial mass="0.1" />
         <visual>
-            <origin xyz="-0.008 0.003 -0.0063" rpy="${-pi/8} ${pi} ${pi}" />
+            <origin xyz="-0.008 0.003 -0.0063" rpy="${-PI/8} ${PI} ${PI}" />
             <geometry>
                 <mesh filename="package://rca_description/meshes/Gripper_1_1.stl"
@@ -140,5 +140,5 @@
         </visual>
         <collision>
-            <origin xyz="-0.008 0.003 -0.0063" rpy="${-pi/8} ${pi} ${pi}" />
+            <origin xyz="-0.008 0.003 -0.0063" rpy="${-PI/8} ${PI} ${PI}" />
             <geometry>
                 <mesh filename="package://rca_description/meshes/Gripper_1_1.stl"
@@ -159,5 +159,5 @@
     </xacro:macro>
     <!-- JOINTS  Virual or fixed-->
-    <joint name="virtual" type="fixed">
+    <joint name="virtual_joint" type="fixed">
         <parent link="world" />
         <child link="base_link" />
@@ -169,5 +169,5 @@
         <child link="base_plate" />
         <axis xyz="0 0 1" />
-        <limit lower="-${pi/2}" upper="${pi/2}" velocity="${velocity}" effort="${effort}" />
+        <limit lower="-${PI/2}" upper="${PI/2}" velocity="${velocity}" effort="${effort}" />
         <origin xyz="0 0 0.129" rpy="0 0 0" />
     </joint>
@@ -176,5 +176,5 @@
         <child link="arm_1" />
         <axis xyz="0 1 0 " />
-        <limit lower="-${pi/4}" upper="${pi/4}"  velocity="${velocity}" effort="${effort}" />
+        <limit lower="-${PI/4}" upper="${PI/4}"  velocity="${velocity}" effort="${effort}" />
         <origin xyz="0.014 0.004 0.04" rpy="0 0 0" />
     </joint>
@@ -183,5 +183,5 @@
         <child link="arm_2" />
         <axis xyz="0 1 0 " />
-        <limit lower="0" upper="${pi/2}"  velocity="${velocity}" effort="${effort}" />
+        <limit lower="-${PI/6}" upper="${PI/2}"  velocity="${velocity}" effort="${effort}" />
         <origin xyz="0 0 0.12" rpy="0 0 0" />
     </joint>
@@ -190,5 +190,5 @@
         <child link="arm_3" />
         <axis xyz="0 0 1 " />
-        <limit lower="-${pi/4}" upper="${pi/4}"  velocity="${velocity}" effort="${effort}" />
+        <limit lower="-${PI/4}" upper="${PI/4}"  velocity="${velocity}" effort="${effort}" />
         <origin xyz="0.0045 0.007 0.09" rpy="0 0 0" />
     </joint>
@@ -197,5 +197,5 @@
         <child link="claw_support" />
         <axis xyz="0 1 0 " />
-        <limit lower="-${pi/4}" upper="${pi/4}"  velocity="${velocity}" effort="${effort}" />
+        <limit lower="-${PI/4}" upper="${PI/4}"  velocity="${velocity}" effort="${effort}" />
         <origin xyz="-0.004 -0.015 0.03" rpy="0 0 0" />
     </joint>
@@ -204,5 +204,5 @@
         <child link="gripper_right" />
         <axis xyz="1 0 0" />
-        <limit lower="-${pi/6}" upper="0"  velocity="${velocity}" effort="${effort}" />
+        <limit lower="-${PI/6}" upper="0"  velocity="${velocity}" effort="${effort}" />
         <origin xyz="0.015 0.004 0.065" rpy="0 0 0" />
     </joint>
@@ -212,5 +212,5 @@
         <child link="gripper_left" />
         <axis xyz="1 0 0" />
-        <limit lower="0" upper="${pi/6}"  velocity="${velocity}" effort="${effort}" />
+        <limit lower="0" upper="${PI/6}"  velocity="${velocity}" effort="${effort}" />
         <origin xyz="0.015 -0.03 0.065" rpy="0 0 0" />
     </joint>

File: rca_description/urdf/ros2_control.xacro (robot description, xacro)
@@ -5,4 +5,24 @@
             <plugin>gazebo_ros2_control/GazeboSystem</plugin>
         </hardware>
+        <!-- ros2_control Gazebo
+        <xacro:if value="$(arg is_sim)">
+            <hardware>
+                <plugin>gazebo_ros2_control/GazeboSystem</plugin>
+            </hardware>
+            <joint name="joint_7">
+                <param name="mimic">joint_6</param>
+                <param name="multiplier">-1</param>
+                <command_interface name="position">
+                    <param name="min">0.0</param>
+                    <param name="max">${PI / 2}</param>
+                </command_interface>
+            </joint>
+        </xacro:if>
+        <xacro:unless value="$(arg is_sim)">
+            <hardware>
+                <plugin>arduinobot_controller/ArduinobotInterface</plugin>
+                <param name="port">/dev/ttyUSB0</param>
+            </hardware>
+        </xacro:unless> -->
         <joint name="joint_1">
             <command_interface name="position">
@@ -21,5 +41,5 @@
         <joint name="joint_3">
             <command_interface name="position">
-                <param name="min">0.0</param>
+                <param name="min">-${PI / 6}</param>
                 <param name="max">${PI / 2}</param>
             </command_interface>
@@ -52,5 +72,5 @@
             <command_interface name="position">
                 <param name="min">0.0</param>
-                <param name="max">${PI/6}</param>
+                <param name="max">${PI / 2}</param>
             </command_interface>
         </joint>
