Commit message: fast fertig

File: rca_description/urdf/rca.urdf.xacro (robot description, xacro)
@@ -1,4 +1,5 @@
 <?xml version="1.0"?>
 <robot xmlns:xacro="http://www.ros.org/wiki/xacro" name="rca">
+    <xacro:arg name="is_sim" default="true"/>
     <!-- Erst Material Laden.. -->
     <xacro:include filename="$(find rca_description)/urdf/material.xacro"/>

File: rca_description/urdf/ros2_control.xacro (robot description, xacro)
@@ -2,8 +2,5 @@
 <robot xmlns:xacro="http://www.ros.org/wiki/xacro" name="rca">
     <ros2_control name="RobotSystem" type="system">
-        <hardware>
-            <plugin>gazebo_ros2_control/GazeboSystem</plugin>
-        </hardware>
-        <!-- ros2_control Gazebo
+        <!-- ros2_control Gazebo -->
         <xacro:if value="$(arg is_sim)">
             <hardware>
@@ -21,8 +18,8 @@
         <xacro:unless value="$(arg is_sim)">
             <hardware>
-                <plugin>arduinobot_controller/ArduinobotInterface</plugin>
+                <plugin>rca_controller/RcaInterface</plugin>
                 <param name="port">/dev/ttyUSB0</param>
             </hardware>
-        </xacro:unless> -->
+        </xacro:unless>
         <joint name="joint_1">
             <command_interface name="position">
@@ -67,12 +64,4 @@
             <state_interface name="position" />
         </joint>
-        <joint name="joint_7">
-            <param name="mimic">joint_6</param>
-            <param name="multiplier">-1</param>
-            <command_interface name="position">
-                <param name="min">0.0</param>
-                <param name="max">${PI / 6}</param>
-            </command_interface>
-        </joint>
     </ros2_control>
 </robot>
