Commit message: in work

File: rca_description/urdf/rca_core.xacro (robot description, xacro)
@@ -67,9 +67,11 @@
             <material name="white" />
         </visual>
-        <origin xyz="0 0.0018 0.035" rpy="${pi/2} 0 ${pi}" />
-        <geometry>
-            <mesh filename="package://rca_description/meshes/Arm_02.stl"
+        <collision>
+            <origin xyz="0 0.0018 0.035" rpy="${pi/2} 0 ${pi}" />
+            <geometry>
+                <mesh filename="package://rca_description/meshes/Arm_02.stl"
                 scale="0.001 0.001 0.001" />
-        </geometry>
+            </geometry>
+        </collision>
     </link>
     <link name="arm_3">
@@ -101,9 +103,11 @@
             <material name="blue" />
         </visual>
-        <origin xyz="0.0095 0.005 0.063" rpy="0 0 ${-pi/2}" />
-        <geometry>
-            <mesh filename="package://rca_description/meshes/Gripper_base.stl"
+        <collision>
+            <origin xyz="0.0095 0.005 0.063" rpy="0 0 ${-pi/2}" />
+            <geometry>
+                <mesh filename="package://rca_description/meshes/Gripper_base.stl"
                 scale="0.001 0.001 0.001" />
-        </geometry>
+            </geometry>
+        </collision>
     </link>
     <link name="gripper_right">
@@ -204,5 +208,5 @@
     </joint>
     <joint name="joint_7" type="revolute">
-        <mimic joint="joint_6" multiplier="-1" offset="0" />
+        <mimic joint="joint_6" multiplier="-1" />
         <parent link="claw_support" />
         <child link="gripper_left" />

Commit message: searching a fail...

File: rca_description/urdf/rca_core.xacro (robot description, xacro)
@@ -150,8 +150,8 @@
     <!-- TRANSMISSION -->
     <xacro:macro name="default_transmission" params="number">
-        <transmission name="transmission_${number}" >
+        <transmission name="transmission_${number}">
             <plugin>transmission_interface/SimpleTransmission</plugin>
-            <actuator name="motor_${number}" roll="actuator1"/>
-            <joint name="joint_${number}" roll="joint1">
+            <actuator name="motor_${number}" role="actuator1"/>
+            <joint name="joint_${number}"    role="joint1">
                 <mechanical_reduction>1.0</mechanical_reduction>
             </joint>
@@ -221,4 +221,3 @@
     <xacro:default_transmission number="5"/>
     <xacro:default_transmission number="6"/>
-    <xacro:default_transmission number="7"/>
 </robot>

File: rca_description/urdf/ros2_control.xacro (robot description, xacro)
@@ -1,4 +1,4 @@
 <?xml version="1.0"?>
-<robot xmlns:xacro="http://www.ros.org/wiki/xacro">
+<robot xmlns:xacro="http://www.ros.org/wiki/xacro" name="rca">
     <xacro:property name="PI" value="3.14159" />
     <ros2_control name="RobotSystem" type="system">
@@ -8,6 +8,6 @@
         <joint name="joint_1">
             <command_interface name="position">
-                <param name="min">${-PI/2}</param>
-                <param name="max">${PI/2}</param>
+                <param name="min">-${PI / 2}</param>
+                <param name="max">${PI / 2}</param>
             </command_interface>
             <state_interface name="position" />
@@ -15,6 +15,6 @@
         <joint name="joint_2">
             <command_interface name="position">
-                <param name="min">${-PI/4}</param>
-                <param name="max">${PI/4}</param>
+                <param name="min">-${PI / 4}</param>
+                <param name="max">${PI / 4}</param>
             </command_interface>
             <state_interface name="position" />
@@ -23,5 +23,5 @@
             <command_interface name="position">
                 <param name="min">0.0</param>
-                <param name="max">${pi/2}</param>
+                <param name="max">${PI / 2}</param>
             </command_interface>
             <state_interface name="position" />
@@ -29,6 +29,6 @@
         <joint name="joint_4">
             <command_interface name="position">
-                <param name="min">${-PI/4}</param>
-                <param name="max">${PI/4}</param>
+                <param name="min">-${PI / 4}</param>
+                <param name="max">${PI / 4}</param>
             </command_interface>
             <state_interface name="position" />
@@ -36,6 +36,6 @@
         <joint name="joint_5">
             <command_interface name="position">
-                <param name="min">${-PI/4}</param>
-                <param name="max">${PI/4}</param>
+                <param name="min">-${PI / 4}</param>
+                <param name="max">${PI / 4}</param>
             </command_interface>
             <state_interface name="position" />
@@ -43,5 +43,5 @@
         <joint name="joint_6">
             <command_interface name="position">
-                <param name="min">${-PI/6}</param>
+                <param name="min">-${PI / 6}</param>
                 <param name="max">0</param>
             </command_interface>
@@ -55,5 +55,4 @@
                 <param name="max">${PI/6}</param>
             </command_interface>
-            <state_interface name="position" />
         </joint>
     </ros2_control>

Commit message: moveit_api_template

File: rca_description/urdf/rca_core.xacro (robot description, xacro)
@@ -169,5 +169,5 @@
         <child link="base_plate" />
         <axis xyz="0 0 1" />
-        <limit lower="-${PI/2}" upper="${PI/2}" velocity="${velocity}" effort="${effort}" />
+        <limit lower="-${PI/4}" upper="${PI/4}" velocity="${velocity}" effort="${effort}" />
         <origin xyz="0 0 0.129" rpy="0 0 0" />
     </joint>
@@ -204,5 +204,5 @@
         <child link="gripper_right" />
         <axis xyz="1 0 0" />
-        <limit lower="-${PI/6}" upper="0"  velocity="${velocity}" effort="${effort}" />
+        <limit lower="-${PI/6}" upper="0.0"  velocity="${velocity}" effort="${effort}" />
         <origin xyz="0.015 0.004 0.065" rpy="0 0 0" />
     </joint>
@@ -212,5 +212,5 @@
         <child link="gripper_left" />
         <axis xyz="1 0 0" />
-        <limit lower="0" upper="${PI/6}"  velocity="${velocity}" effort="${effort}" />
+        <limit lower="0.0" upper="${PI/6}"  velocity="${velocity}" effort="${effort}" />
         <origin xyz="0.015 -0.03 0.065" rpy="0 0 0" />
     </joint>

File: rca_description/urdf/ros2_control.xacro (robot description, xacro)
@@ -27,6 +27,6 @@
         <joint name="joint_1">
             <command_interface name="position">
-                <param name="min">-${PI / 2}</param>
-                <param name="max">${PI / 2}</param>
+                <param name="min">-${PI / 4}</param>  <!-- 0,785375-->
+                <param name="max">${PI / 4}</param>
             </command_interface>
             <state_interface name="position" />
@@ -41,6 +41,6 @@
         <joint name="joint_3">
             <command_interface name="position">
-                <param name="min">-${PI / 6}</param>
-                <param name="max">${PI / 2}</param>
+                <param name="min">-${PI / 6}</param> <!-- -0,52358-->
+                <param name="max">${PI / 2}</param>  <!--  1,57075 -->
             </command_interface>
             <state_interface name="position" />
@@ -72,5 +72,5 @@
             <command_interface name="position">
                 <param name="min">0.0</param>
-                <param name="max">${PI / 2}</param>
+                <param name="max">${PI / 6}</param>
             </command_interface>
         </joint>

Commit message: setting start points

File: rca_description/urdf/rca_core.xacro (robot description, xacro)
@@ -169,5 +169,5 @@
         <child link="base_plate" />
         <axis xyz="0 0 1" />
-        <limit lower="-${PI/4}" upper="${PI/4}" velocity="${velocity}" effort="${effort}" />
+        <limit lower="-${PI/2}" upper="${PI/2}" velocity="${velocity}" effort="${effort}" />
         <origin xyz="0 0 0.129" rpy="0 0 0" />
     </joint>
@@ -176,5 +176,5 @@
         <child link="arm_1" />
         <axis xyz="0 1 0 " />
-        <limit lower="-${PI/4}" upper="${PI/4}"  velocity="${velocity}" effort="${effort}" />
+        <limit lower="-${PI/2}" upper="${PI/2}"  velocity="${velocity}" effort="${effort}" />
         <origin xyz="0.014 0.004 0.04" rpy="0 0 0" />
     </joint>
@@ -183,6 +183,6 @@
         <child link="arm_2" />
         <axis xyz="0 1 0 " />
-        <limit lower="-${PI/6}" upper="${PI/2}"  velocity="${velocity}" effort="${effort}" />
-        <origin xyz="0 0 0.12" rpy="0 0 0" />
+        <limit lower="-${PI/2}" upper="${PI/2}"  velocity="${velocity}" effort="${effort}" />
+        <origin xyz="0 0 0.12" rpy="0 ${PI/4} 0" />
     </joint>
     <joint name="joint_4" type="revolute">

File: rca_description/urdf/ros2_control.xacro (robot description, xacro)
@@ -24,6 +24,6 @@
         <joint name="joint_1">
             <command_interface name="position">
-                <param name="min">-${PI / 4}</param>  <!-- 0,785375-->
-                <param name="max">${PI / 4}</param>
+                <param name="min">-${PI / 2}</param>
+                <param name="max">${PI / 2}</param>
             </command_interface>
             <state_interface name="position" />
@@ -31,6 +31,6 @@
         <joint name="joint_2">
             <command_interface name="position">
-                <param name="min">-${PI / 4}</param>
-                <param name="max">${PI / 4}</param>
+                <param name="min">-${PI / 2}</param>
+                <param name="max">${PI / 2}</param>
             </command_interface>
             <state_interface name="position" />
@@ -38,6 +38,6 @@
         <joint name="joint_3">
             <command_interface name="position">
-                <param name="min">-${PI / 6}</param> <!-- -0,52358-->
-                <param name="max">${PI / 2}</param>  <!--  1,57075 -->
+                <param name="min">-${PI / 2}</param>
+                <param name="max">${PI / 2}</param>
             </command_interface>
             <state_interface name="position" />
