Commit message: ros2 control works

File: rca_description/urdf/gazebo.xacro (robot description, xacro)
@@ -5,6 +5,30 @@
             <robot_param>robot_description</robot_param>
             <robot_param_node>robot_state_publisher</robot_param_node>
-            <parameters></parameters>
+            <parameters>$(find rca_controller)/config/rca_controllers.yaml</parameters>
         </plugin>
     </gazebo>
+    <gazebo reference="base_link">
+        <material>Gazebo/Black</material>
+    </gazebo>
+    <gazebo reference="base_plate">
+        <material>Gazebo/Blue</material>
+    </gazebo>
+    <gazebo reference="arm_1">
+        <material>Gazebo/White</material>
+    </gazebo>
+    <gazebo reference="arm_2">
+        <material>Gazebo/White</material>
+    </gazebo>
+    <gazebo reference="arm_3">
+        <material>Gazebo/White</material>
+    </gazebo>
+    <gazebo reference="claw_support">
+        <material>Gazebo/Black</material>
+    </gazebo>
+    <gazebo reference="gripper_right">
+        <material>Gazebo/Green</material>
+    </gazebo>
+    <gazebo reference="gripper_left">
+        <material>Gazebo/Red</material>
+    </gazebo>
 </robot>

File: rca_description/urdf/material.xacro (robot description, xacro)
@@ -1,4 +1,6 @@
 <?xml version="1.0"?>
 <robot xmlns:xacro="http://www.ros.org/wiki/xacro" >
+    <xacro:property name="effort" value="30.0" />
+    <xacro:property name="velocity" value="10.0" />
     <material name="white">
         <color rgba="1 1 1 0.8"/>
@@ -8,10 +10,10 @@
     </material>
     <!-- Inertial-->
-    <xacro:macro name="default_inertial" params="mass"> <!-- <xacro:default_inertial mass="1"/> -->
+    <xacro:macro name="default_inertial" params="mass"> <!-- <xacro:default_inertial mass="1.0"/> -->
         <inertial>
             <mass value="${mass}" />
-            <inertia ixx="1.0" ixy="0.0" ixz="0.0"
-                     iyy="1.0" iyz="0.0"
-                     izz="1.0" />
+            <inertia ixx="0.0001" ixy="0.0" ixz="0.0"
+                     iyy="0.0001" iyz="0.0"
+                     izz="0.0001" />
         </inertial>
     </xacro:macro>

File: rca_description/urdf/rca.urdf.xacro (robot description, xacro)
@@ -1,10 +1,8 @@
 <?xml version="1.0"?>
 <robot xmlns:xacro="http://www.ros.org/wiki/xacro" name="rca">
-    <!-- Erst Material Laden -->
+    <!-- Erst Material Laden.. -->
     <xacro:include filename="material.xacro"/>
-    <!--  dann die STL Files zum visualisieren -->
-    <xacro:include filename="robot.xacro"/>
-    <!-- Laden der Gelenke -->
-    <xacro:include filename="joints.xacro"/>
+    <!--  ..dann die STL Files zum visualisieren -->
+    <xacro:include filename="rca_core.xacro"/>
     <!-- Gazebo plugins -->
     <xacro:include filename="gazebo.xacro"/>

File: rca_description/urdf/rca_core.xacro (robot description, xacro)
@@ -143,3 +143,78 @@
         </collision>
     </link>
+    <!-- JOINTS -->
+    <!-- TRANSMISSION -->
+    <xacro:macro name="default_transmission" params="number">
+        <transmission name="transmission_${number}" >
+            <plugin>transmission_interface/SimpleTransmission</plugin>
+            <actuator name="motor_${number}" roll="actuator1"/>
+            <joint name="joint_${number}" roll="joint1">
+                <mechanical_reduction>1.0</mechanical_reduction>
+            </joint>
+        </transmission>
+    </xacro:macro>
+    <!-- JOINTS  Virual or fixed-->
+    <joint name="virtual" type="fixed">
+        <parent link="world" />
+        <child link="base_link" />
+        <origin xyz="0.0 0.0 0.0" rpy="0.0 0.0 0.0" />
+    </joint>
+    <!-- JOINTS  Revolute-->
+    <joint name="joint_1" type="revolute">
+        <parent link="base_link" />
+        <child link="base_plate" />
+        <axis xyz="0 0 1" />
+        <limit lower="${-pi/2}" upper="${pi/2}" velocity="${velocity}" effort="${effort}" />
+        <origin xyz="0 0 0.129" rpy="0 0 0" />
+    </joint>
+    <joint name="joint_2" type="revolute">
+        <parent link="base_plate" />
+        <child link="arm_1" />
+        <axis xyz="0 1 0 " />
+        <limit lower="${-pi/4}" upper="${pi/4}"  velocity="${velocity}" effort="${effort}" />
+        <origin xyz="0.014 0.004 0.04" rpy="0 0 0" />
+    </joint>
+    <joint name="joint_3" type="revolute">
+        <parent link="arm_1" />
+        <child link="arm_2" />
+        <axis xyz="0 1 0 " />
+        <limit lower="0" upper="${pi/2}"  velocity="${velocity}" effort="${effort}" />
+        <origin xyz="0 0 0.12" rpy="0 0 0" />
+    </joint>
+    <joint name="joint_4" type="revolute">
+        <parent link="arm_2" />
+        <child link="arm_3" />
+        <axis xyz="0 0 1 " />
+        <limit lower="${-pi/4}" upper="${pi/4}"  velocity="${velocity}" effort="${effort}" />
+        <origin xyz="0.0045 0.007 0.09" rpy="0 0 0" />
+    </joint>
+    <joint name="joint_5" type="revolute">
+        <parent link="arm_3" />
+        <child link="claw_support" />
+        <axis xyz="0 1 0 " />
+        <limit lower="${-pi/4}" upper="${pi/4}"  velocity="${velocity}" effort="${effort}" />
+        <origin xyz="-0.004 -0.015 0.03" rpy="0 0 0" />
+    </joint>
+    <joint name="joint_6" type="revolute">
+        <parent link="claw_support" />
+        <child link="gripper_right" />
+        <axis xyz="1 0 0" />
+        <limit lower="${-pi/6}" upper="0"  velocity="${velocity}" effort="${effort}" />
+        <origin xyz="0.015 0.004 0.065" rpy="0 0 0" />
+    </joint>
+    <joint name="joint_7" type="revolute">
+        <mimic joint="joint_6" multiplier="-1" offset="0" />
+        <parent link="claw_support" />
+        <child link="gripper_left" />
+        <axis xyz="1 0 0" />
+        <limit lower="0" upper="${pi/6}"  velocity="${velocity}" effort="${effort}" />
+        <origin xyz="0.015 -0.03 0.065" rpy="0 0 0" />
+    </joint>
+    <xacro:default_transmission number="1"/>
+    <xacro:default_transmission number="2"/>
+    <xacro:default_transmission number="3"/>
+    <xacro:default_transmission number="4"/>
+    <xacro:default_transmission number="5"/>
+    <xacro:default_transmission number="6"/>
+    <xacro:default_transmission number="7"/>
 </robot>

File: rca_description/urdf/ros2_control.xacro (robot description, xacro)
@@ -4,5 +4,5 @@
     <ros2_control name="RobotSystem" type="system">
         <hardware>
-            <plugin> gazebo_ros2_control/GazeboSystem </plugin>
+            <plugin>gazebo_ros2_control/GazeboSystem</plugin>
         </hardware>
         <joint name="joint_1">
@@ -15,6 +15,6 @@
         <joint name="joint_2">
             <command_interface name="position">
-                <param name="min">${-PI/2}</param>
-                <param name="max">${PI/2}</param>
+                <param name="min">${-PI/4}</param>
+                <param name="max">${PI/4}</param>
             </command_interface>
             <state_interface name="position" />
@@ -22,6 +22,6 @@
         <joint name="joint_3">
             <command_interface name="position">
-                <param name="min">-0.1</param>
-                <param name="max">2.77</param>
+                <param name="min">0.0</param>
+                <param name="max">${pi/2}</param>
             </command_interface>
             <state_interface name="position" />

Commit message: dont know

File: rca_description/urdf/gazebo.xacro (robot description, xacro)
@@ -1,4 +1,4 @@
 <?xml version="1.0"?>
-<robot xmlns:xacro="http://www.ros.org/wiki/xacro" >
+<robot xmlns:xacro="http://www.ros.org/wiki/xacro" name="rca">
     <gazebo>
         <plugin filename="libgazebo_ros2_control.so" name="gazebo_ros2_control" >

File: rca_description/urdf/material.xacro (robot description, xacro)
@@ -1,4 +1,5 @@
 <?xml version="1.0"?>
 <robot xmlns:xacro="http://www.ros.org/wiki/xacro" >
+    <xacro:property name="PI" value="3.14159" />
     <xacro:property name="effort" value="30.0" />
     <xacro:property name="velocity" value="10.0" />

File: rca_description/urdf/rca.urdf.xacro (robot description, xacro)
@@ -2,10 +2,10 @@
 <robot xmlns:xacro="http://www.ros.org/wiki/xacro" name="rca">
     <!-- Erst Material Laden.. -->
-    <xacro:include filename="material.xacro"/>
+    <xacro:include filename="$(find rca_description)/urdf/material.xacro"/>
     <!--  ..dann die STL Files zum visualisieren -->
-    <xacro:include filename="rca_core.xacro"/>
+    <xacro:include filename="$(find rca_description)/urdf/rca_core.xacro"/>
     <!-- Gazebo plugins -->
-    <xacro:include filename="gazebo.xacro"/>
+    <xacro:include filename="$(find rca_description)/urdf/gazebo.xacro"/>
     <!-- ROS2_Control -->
-    <xacro:include filename="ros2_control.xacro"/>
+    <xacro:include filename="$(find rca_description)/urdf/ros2_control.xacro"/>
 </robot>

File: rca_description/urdf/rca_core.xacro (robot description, xacro)
@@ -1,4 +1,4 @@
 <?xml version="1.0"?>
-<robot xmlns:xacro="http://www.ros.org/wiki/xacro">
+<robot xmlns:xacro="http://www.ros.org/wiki/xacro" name="rca">
     <!-- LINKS -->
     <link name="world" />
@@ -169,5 +169,5 @@
         <child link="base_plate" />
         <axis xyz="0 0 1" />
-        <limit lower="${-pi/2}" upper="${pi/2}" velocity="${velocity}" effort="${effort}" />
+        <limit lower="-${pi/2}" upper="${pi/2}" velocity="${velocity}" effort="${effort}" />
         <origin xyz="0 0 0.129" rpy="0 0 0" />
     </joint>
@@ -176,5 +176,5 @@
         <child link="arm_1" />
         <axis xyz="0 1 0 " />
-        <limit lower="${-pi/4}" upper="${pi/4}"  velocity="${velocity}" effort="${effort}" />
+        <limit lower="-${pi/4}" upper="${pi/4}"  velocity="${velocity}" effort="${effort}" />
         <origin xyz="0.014 0.004 0.04" rpy="0 0 0" />
     </joint>
@@ -190,5 +190,5 @@
         <child link="arm_3" />
         <axis xyz="0 0 1 " />
-        <limit lower="${-pi/4}" upper="${pi/4}"  velocity="${velocity}" effort="${effort}" />
+        <limit lower="-${pi/4}" upper="${pi/4}"  velocity="${velocity}" effort="${effort}" />
         <origin xyz="0.0045 0.007 0.09" rpy="0 0 0" />
     </joint>
@@ -197,5 +197,5 @@
         <child link="claw_support" />
         <axis xyz="0 1 0 " />
-        <limit lower="${-pi/4}" upper="${pi/4}"  velocity="${velocity}" effort="${effort}" />
+        <limit lower="-${pi/4}" upper="${pi/4}"  velocity="${velocity}" effort="${effort}" />
         <origin xyz="-0.004 -0.015 0.03" rpy="0 0 0" />
     </joint>
@@ -204,5 +204,5 @@
         <child link="gripper_right" />
         <axis xyz="1 0 0" />
-        <limit lower="${-pi/6}" upper="0"  velocity="${velocity}" effort="${effort}" />
+        <limit lower="-${pi/6}" upper="0"  velocity="${velocity}" effort="${effort}" />
         <origin xyz="0.015 0.004 0.065" rpy="0 0 0" />
     </joint>

File: rca_description/urdf/ros2_control.xacro (robot description, xacro)
@@ -1,5 +1,4 @@
 <?xml version="1.0"?>
 <robot xmlns:xacro="http://www.ros.org/wiki/xacro" name="rca">
-    <xacro:property name="PI" value="3.14159" />
     <ros2_control name="RobotSystem" type="system">
         <hardware>

Commit message: changed color

File: rca_description/urdf/gazebo.xacro (robot description, xacro)
@@ -9,23 +9,23 @@
     </gazebo>
     <gazebo reference="base_link">
+        <material>Gazebo/Red</material>
+    </gazebo>
+    <gazebo reference="base_plate">
         <material>Gazebo/Black</material>
     </gazebo>
-    <gazebo reference="base_plate">
-        <material>Gazebo/Blue</material>
-    </gazebo>
     <gazebo reference="arm_1">
-        <material>Gazebo/White</material>
+        <material>Gazebo/Red</material>
     </gazebo>
     <gazebo reference="arm_2">
-        <material>Gazebo/White</material>
+        <material>Gazebo/Red</material>
     </gazebo>
     <gazebo reference="arm_3">
-        <material>Gazebo/White</material>
+        <material>Gazebo/Red</material>
     </gazebo>
     <gazebo reference="claw_support">
-        <material>Gazebo/Black</material>
+        <material>Gazebo/Red</material>
     </gazebo>
     <gazebo reference="gripper_right">
-        <material>Gazebo/Green</material>
+        <material>Gazebo/Red</material>
     </gazebo>
     <gazebo reference="gripper_left">

File: rca_description/urdf/material.xacro (robot description, xacro)
@@ -10,4 +10,10 @@
         <color rgba="0.0 0.0 1.0 0.8"/>
     </material>
+    <material name="black">
+        <color rgba="0.0 0.0 0.0 1.0"/>
+    </material>
+    <material name="red">
+        <color rgba="1.0 0.0 0.0 0.8"/>
+    </material>
     <!-- Inertial-->
     <xacro:macro name="default_inertial" params="mass"> <!-- <xacro:default_inertial mass="1.0"/> -->

File: rca_description/urdf/rca_core.xacro (robot description, xacro)
@@ -29,5 +29,5 @@
                     scale="0.001 0.001 0.001" />
             </geometry>
-            <material name="blue" />
+            <material name="black" />
         </visual>
         <collision>
@@ -47,5 +47,5 @@
                     scale="0.001 0.001 0.001" />
             </geometry>
-            <material name="white" />
+            <material name="red" />
         </visual>
         <collision>
@@ -65,5 +65,5 @@
                     scale="0.001 0.001 0.001" />
             </geometry>
-            <material name="white" />
+            <material name="red" />
         </visual>
         <collision>
@@ -83,5 +83,5 @@
                     scale="0.001 0.001 0.001" />
             </geometry>
-            <material name="white" />
+            <material name="red" />
         </visual>
         <collision>
@@ -119,5 +119,5 @@
                     scale="0.001 0.001 0.001" />
             </geometry>
-            <material name="white" />
+            <material name="red" />
         </visual>
         <collision>
@@ -137,5 +137,5 @@
                     scale="0.001 0.001 0.001" />
             </geometry>
-            <material name="white" />
+            <material name="red" />
         </visual>
         <collision>
